Commit message: fix: run mujoco headless via xvfb and load mjcf from urdf param

File: src/fm_control/urdf/openarm.ros2_control.xacro (robot description, xacro)
@@ -30,4 +30,7 @@
       <hardware>
         <plugin>mujoco_ros2_control/MujocoSystemInterface</plugin>
+        <!-- MujocoSystemInterface reads the MJCF from this URDF param.
+             mujoco_model_path is set by the top-level xacro. -->
+        <param name="mujoco_model">${mujoco_model_path}</param>
       </hardware>
     </xacro:if>

File: src/fm_control/urdf/openarm.sim.urdf.xacro (robot description, xacro)
@@ -23,4 +23,9 @@
   <xacro:arg name="isaac_joint_commands_topic" default="/isaac_joint_commands"/>
   <xacro:arg name="isaac_joint_states_topic" default="/isaac_joint_states"/>
+  <!-- MJCF the MuJoCo backend loads. MujocoSystemInterface reads it from this URDF
+       <param>, not a node param. Defaults to the vendored v2 bimanual model
+       (in-container path; src/external is gitignored, mounted at /ws). -->
+  <xacro:arg name="mujoco_model" default="/ws/src/external/openarm_mujoco/v2/openarm_bimanual.xml"/>
+  <xacro:property name="mujoco_model_path" value="$(arg mujoco_model)"/>
   <!-- Controllers file the Gazebo gz_ros2_control plugin loads into its embedded
        controller_manager. Only used by the gazebo backend. -->
