Commit message: feat: actuate left arm in sim

File: src/fm_control/urdf/g1.ros2_control.xacro (robot description, xacro)
@@ -1,8 +1,10 @@
 <?xml version="1.0"?>
 <!--
-First Motive ros2_control for the Unitree G1-D right arm (7 joints).
-One <ros2_control> system for the right arm only — waist, legs, left arm, and the
-wheeled base are left unactuated (they hold at zero via robot_state_publisher in
-sim). Only the <hardware> System plugin swaps, selected by `sim_backend`:
+First Motive ros2_control for the Unitree G1-D arms (left + right, 7 joints each).
+One <ros2_control> system holds both arms; two joint_trajectory_controllers each
+claim their 7 joints (g1_right_arm_controller, g1_left_arm_controller). The waist,
+legs, hands, and the wheeled base are left unactuated here (they hold at zero via
+robot_state_publisher in sim). Only the <hardware> System plugin swaps, selected by
+`sim_backend`:
   mock    -> mock_components/GenericSystem               (no sim; perfect state echo)
   mujoco  -> mujoco_ros2_control/MujocoSystemInterface   (CPU)
@@ -10,12 +12,10 @@
   isaac   -> topic_based_ros2_control/TopicBasedSystem   (Isaac Sim over ROS topics)
 There is deliberately NO `real` ros2_control plugin: no hardware interface exists for
-the G1 upstream. The real arm is driven by the Servo->arm_sdk bridge (a 50 Hz
+the G1 upstream. The real arms are driven by the Servo->arm_sdk bridge (a 50 Hz
 unitree_hg/LowCmd loop on rt/arm_sdk), which replaces the controller + hardware at
 runtime — so for sim_backend=real this macro emits no <ros2_control> at all, leaving
 the description geometry-only for robot_state_publisher. See the bridge node.
-Joint names match the vendored g1_d URDF right arm exactly:
-right_shoulder_pitch_joint, right_shoulder_roll_joint, right_shoulder_yaw_joint,
-right_elbow_joint, right_wrist_roll_joint, right_wrist_pitch_joint,
-right_wrist_yaw_joint (arm_sdk motor_cmd indices 22..28).
+Joint names match the vendored g1_d URDF arms exactly. arm_sdk motor_cmd indices:
+right arm 22..28, left arm 15..21 (unitree_sdk2 JointIndex enum).
 -->
 <robot xmlns:xacro="http://www.ros.org/wiki/xacro">
@@ -67,11 +67,11 @@
     </joint>
   </xacro:macro>
-  <!-- The 7-joint right-arm system, emitted for sim backends only. -->
-  <xacro:macro name="g1_right_arm_system"
+  <!-- The 14-joint dual-arm system, emitted for sim backends only. -->
+  <xacro:macro name="g1_arm_system"
       params="sim_backend mujoco_model_path:=''
               isaac_joint_commands_topic:=/isaac_joint_commands
               isaac_joint_states_topic:=/isaac_joint_states">
     <xacro:unless value="${sim_backend == 'real'}">
-      <ros2_control name="g1_right_arm_system" type="system">
+      <ros2_control name="g1_arm_system" type="system">
         <xacro:g1_backend_hardware
             sim_backend="${sim_backend}"
@@ -86,7 +86,14 @@
         <xacro:g1_arm_joint joint_name="right_wrist_pitch_joint"/>
         <xacro:g1_arm_joint joint_name="right_wrist_yaw_joint"/>
+        <xacro:g1_arm_joint joint_name="left_shoulder_pitch_joint"/>
+        <xacro:g1_arm_joint joint_name="left_shoulder_roll_joint"/>
+        <xacro:g1_arm_joint joint_name="left_shoulder_yaw_joint"/>
+        <xacro:g1_arm_joint joint_name="left_elbow_joint"/>
+        <xacro:g1_arm_joint joint_name="left_wrist_roll_joint"/>
+        <xacro:g1_arm_joint joint_name="left_wrist_pitch_joint"/>
+        <xacro:g1_arm_joint joint_name="left_wrist_yaw_joint"/>
       </ros2_control>
     </xacro:unless>
-    <!-- real: no ros2_control; the Servo->arm_sdk bridge drives the arm at runtime. -->
+    <!-- real: no ros2_control; the Servo->arm_sdk bridge drives the arms at runtime. -->
   </xacro:macro>
 </robot>

File: src/fm_control/urdf/g1.sim.urdf.xacro (robot description, xacro)
@@ -1,11 +1,11 @@
 <?xml version="1.0" encoding="utf-8"?>
 <!--
-First Motive G1-D description with a backend-selectable ros2_control System for the
-right arm.
+First Motive G1-D description with a backend-selectable ros2_control System for both
+arms.
 This merges the vendored Unitree G1-D geometry (the flat URDF installed into
-fm_description's share) and injects a <ros2_control> system that actuates the 7
-right-arm joints, selected by `sim_backend`. The wheeled base, waist, legs, and left
-arm are not actuated — in sim they hold at zero through robot_state_publisher. The
-G1-D is a single fixed configuration, so there is no preset arg.
+fm_description's share) and injects a <ros2_control> system that actuates the 14
+arm joints (7 per arm), selected by `sim_backend`. The wheeled base, waist, legs, and
+hands are not actuated here — in sim they hold at zero through robot_state_publisher.
+The G1-D is a single fixed configuration, so there is no preset arg.
 For sim_backend=real no ros2_control is emitted: the Servo->arm_sdk bridge drives the
 arm out-of-band (see g1.ros2_control.xacro). The description stays geometry-only so
@@ -33,5 +33,5 @@
   <xacro:include filename="$(find fm_description)/g1_d_description/g1_d.urdf"/>
   <xacro:include filename="$(find fm_control)/urdf/g1.ros2_control.xacro"/>
-  <xacro:g1_right_arm_system
+  <xacro:g1_arm_system
       sim_backend="$(arg sim_backend)"
       mujoco_model_path="${mujoco_model_path}"

Commit message: feat: drive wheelbase from cmd_vel

File: src/fm_control/urdf/g1.ros2_control.xacro (robot description, xacro)
@@ -1,10 +1,11 @@
 <?xml version="1.0"?>
 <!--
-First Motive ros2_control for the Unitree G1-D arms (left + right, 7 joints each).
-One <ros2_control> system holds both arms; two joint_trajectory_controllers each
-claim their 7 joints (g1_right_arm_controller, g1_left_arm_controller). The waist,
-legs, hands, and the wheeled base are left unactuated here (they hold at zero via
-robot_state_publisher in sim). Only the <hardware> System plugin swaps, selected by
-`sim_backend`:
+First Motive ros2_control for the Unitree G1-D arms + wheeled base.
+One <ros2_control> system holds both arms (7 joints each) and the two drive wheels.
+Two joint_trajectory_controllers each claim an arm's 7 joints (g1_right_arm_controller,
+g1_left_arm_controller); a diff_drive_controller claims the two wheels' velocity
+interface (g1_base_controller). The waist, legs, and hands are left unactuated here
+(they hold at zero via robot_state_publisher in sim). Only the <hardware> System plugin
+swaps, selected by `sim_backend`:
   mock    -> mock_components/GenericSystem               (no sim; perfect state echo)
   mujoco  -> mujoco_ros2_control/MujocoSystemInterface   (CPU)
@@ -13,9 +14,11 @@
 There is deliberately NO `real` ros2_control plugin: no hardware interface exists for
 the G1 upstream. The real arms are driven by the Servo->arm_sdk bridge (a 50 Hz
-unitree_hg/LowCmd loop on rt/arm_sdk), which replaces the controller + hardware at
-runtime — so for sim_backend=real this macro emits no <ros2_control> at all, leaving
-the description geometry-only for robot_state_publisher. See the bridge node.
-Joint names match the vendored g1_d URDF arms exactly. arm_sdk motor_cmd indices:
-right arm 22..28, left arm 15..21 (unitree_sdk2 JointIndex enum).
+unitree_hg/LowCmd loop on rt/arm_sdk) and the real base by g1_base_teleop (Twist ->
+AGV Move RPC), which replace the controller + hardware at runtime — so for
+sim_backend=real this macro emits no <ros2_control> at all, leaving the description
+geometry-only for robot_state_publisher. See the bridge nodes.
+Joint names match the vendored g1_d URDF exactly. arm_sdk motor_cmd indices: right arm
+22..28, left arm 15..21 (unitree_sdk2 JointIndex enum). The wheels (Left_Wheel_Joint,
+Right_Wheel_Joint) are velocity-controlled in sim only.
 -->
 <robot xmlns:xacro="http://www.ros.org/wiki/xacro">
@@ -67,11 +70,25 @@
     </joint>
   </xacro:macro>
-  <!-- The 14-joint dual-arm system, emitted for sim backends only. -->
-  <xacro:macro name="g1_arm_system"
+  <!-- One drive wheel: velocity command + position/velocity state, claimed by the
+       diff_drive_controller. -->
+  <xacro:macro name="g1_wheel_joint" params="joint_name">
+    <joint name="${joint_name}">
+      <command_interface name="velocity"/>
+      <state_interface name="position">
+        <param name="initial_value">0.0</param>
+      </state_interface>
+      <state_interface name="velocity">
+        <param name="initial_value">0.0</param>
+      </state_interface>
+    </joint>
+  </xacro:macro>
+  <!-- The dual-arm + wheeled-base system (14 arm joints + 2 wheels), emitted for sim
+       backends only. -->
+  <xacro:macro name="g1_system"
       params="sim_backend mujoco_model_path:=''
               isaac_joint_commands_topic:=/isaac_joint_commands
               isaac_joint_states_topic:=/isaac_joint_states">
     <xacro:unless value="${sim_backend == 'real'}">
-      <ros2_control name="g1_arm_system" type="system">
+      <ros2_control name="g1_system" type="system">
         <xacro:g1_backend_hardware
             sim_backend="${sim_backend}"
@@ -93,7 +110,10 @@
         <xacro:g1_arm_joint joint_name="left_wrist_pitch_joint"/>
         <xacro:g1_arm_joint joint_name="left_wrist_yaw_joint"/>
+        <xacro:g1_wheel_joint joint_name="Left_Wheel_Joint"/>
+        <xacro:g1_wheel_joint joint_name="Right_Wheel_Joint"/>
       </ros2_control>
     </xacro:unless>
-    <!-- real: no ros2_control; the Servo->arm_sdk bridge drives the arms at runtime. -->
+    <!-- real: no ros2_control; the Servo->arm_sdk bridge drives the arms and
+         g1_base_teleop drives the base at runtime. -->
   </xacro:macro>
 </robot>

File: src/fm_control/urdf/g1.sim.urdf.xacro (robot description, xacro)
@@ -5,7 +5,8 @@
 This merges the vendored Unitree G1-D geometry (the flat URDF installed into
 fm_description's share) and injects a <ros2_control> system that actuates the 14
-arm joints (7 per arm), selected by `sim_backend`. The wheeled base, waist, legs, and
-hands are not actuated here — in sim they hold at zero through robot_state_publisher.
-The G1-D is a single fixed configuration, so there is no preset arg.
+arm joints (7 per arm) plus the two drive wheels, selected by `sim_backend`. The
+waist, legs, and hands are not actuated here — in sim they hold at zero through
+robot_state_publisher. The G1-D is a single fixed configuration, so there is no
+preset arg.
 For sim_backend=real no ros2_control is emitted: the Servo->arm_sdk bridge drives the
 arm out-of-band (see g1.ros2_control.xacro). The description stays geometry-only so
@@ -33,5 +34,5 @@
   <xacro:include filename="$(find fm_description)/g1_d_description/g1_d.urdf"/>
   <xacro:include filename="$(find fm_control)/urdf/g1.ros2_control.xacro"/>
-  <xacro:g1_arm_system
+  <xacro:g1_system
       sim_backend="$(arg sim_backend)"
       mujoco_model_path="${mujoco_model_path}"

Commit message: feat: actuate dex3 hands in sim

File: src/fm_control/urdf/g1.ros2_control.xacro (robot description, xacro)
@@ -1,11 +1,12 @@
 <?xml version="1.0"?>
 <!--
-First Motive ros2_control for the Unitree G1-D arms + wheeled base.
-One <ros2_control> system holds both arms (7 joints each) and the two drive wheels.
-Two joint_trajectory_controllers each claim an arm's 7 joints (g1_right_arm_controller,
-g1_left_arm_controller); a diff_drive_controller claims the two wheels' velocity
-interface (g1_base_controller). The waist, legs, and hands are left unactuated here
-(they hold at zero via robot_state_publisher in sim). Only the <hardware> System plugin
-swaps, selected by `sim_backend`:
+First Motive ros2_control for the Unitree G1-D arms + Dex3 hands + wheeled base.
+One <ros2_control> system holds both arms (7 joints each), both Dex3 hands (7 finger
+joints each), and the two drive wheels. A joint_trajectory_controller claims each arm
+(g1_right_arm_controller, g1_left_arm_controller) and each hand (g1_right_hand_controller,
+g1_left_hand_controller); a diff_drive_controller claims the two wheels' velocity
+interface (g1_base_controller). The waist and legs are left unactuated here (they hold
+at zero via robot_state_publisher in sim). Only the <hardware> System plugin swaps,
+selected by `sim_backend`:
   mock    -> mock_components/GenericSystem               (no sim; perfect state echo)
   mujoco  -> mujoco_ros2_control/MujocoSystemInterface   (CPU)
@@ -52,7 +53,8 @@
     </xacro:if>
   </xacro:macro>
-  <!-- One joint: position/velocity/effort command + state, uniform across the sim
-       backends so the controller set never changes. -->
-  <xacro:macro name="g1_arm_joint" params="joint_name">
+  <!-- One position-controlled joint: position/velocity/effort command + state, uniform
+       across the sim backends so the controller set never changes. Used for both arm
+       joints and the Dex3 hand finger joints. -->
+  <xacro:macro name="g1_position_joint" params="joint_name">
     <joint name="${joint_name}">
       <command_interface name="position"/>
@@ -83,6 +85,6 @@
     </joint>
   </xacro:macro>
-  <!-- The dual-arm + wheeled-base system (14 arm joints + 2 wheels), emitted for sim
-       backends only. -->
+  <!-- The full G1-D control system (14 arm joints + 14 hand joints + 2 wheels), emitted
+       for sim backends only. -->
   <xacro:macro name="g1_system"
       params="sim_backend mujoco_model_path:=''
@@ -96,20 +98,37 @@
             isaac_joint_commands_topic="${isaac_joint_commands_topic}"
             isaac_joint_states_topic="${isaac_joint_states_topic}" />
-        <xacro:g1_arm_joint joint_name="right_shoulder_pitch_joint"/>
-        <xacro:g1_arm_joint joint_name="right_shoulder_roll_joint"/>
-        <xacro:g1_arm_joint joint_name="right_shoulder_yaw_joint"/>
-        <xacro:g1_arm_joint joint_name="right_elbow_joint"/>
-        <xacro:g1_arm_joint joint_name="right_wrist_roll_joint"/>
-        <xacro:g1_arm_joint joint_name="right_wrist_pitch_joint"/>
-        <xacro:g1_arm_joint joint_name="right_wrist_yaw_joint"/>
-        <xacro:g1_arm_joint joint_name="left_shoulder_pitch_joint"/>
-        <xacro:g1_arm_joint joint_name="left_shoulder_roll_joint"/>
-        <xacro:g1_arm_joint joint_name="left_shoulder_yaw_joint"/>
-        <xacro:g1_arm_joint joint_name="left_elbow_joint"/>
-        <xacro:g1_arm_joint joint_name="left_wrist_roll_joint"/>
-        <xacro:g1_arm_joint joint_name="left_wrist_pitch_joint"/>
-        <xacro:g1_arm_joint joint_name="left_wrist_yaw_joint"/>
+        <xacro:g1_position_joint joint_name="right_shoulder_pitch_joint"/>
+        <xacro:g1_position_joint joint_name="right_shoulder_roll_joint"/>
+        <xacro:g1_position_joint joint_name="right_shoulder_yaw_joint"/>
+        <xacro:g1_position_joint joint_name="right_elbow_joint"/>
+        <xacro:g1_position_joint joint_name="right_wrist_roll_joint"/>
+        <xacro:g1_position_joint joint_name="right_wrist_pitch_joint"/>
+        <xacro:g1_position_joint joint_name="right_wrist_yaw_joint"/>
+        <xacro:g1_position_joint joint_name="left_shoulder_pitch_joint"/>
+        <xacro:g1_position_joint joint_name="left_shoulder_roll_joint"/>
+        <xacro:g1_position_joint joint_name="left_shoulder_yaw_joint"/>
+        <xacro:g1_position_joint joint_name="left_elbow_joint"/>
+        <xacro:g1_position_joint joint_name="left_wrist_roll_joint"/>
+        <xacro:g1_position_joint joint_name="left_wrist_pitch_joint"/>
+        <xacro:g1_position_joint joint_name="left_wrist_yaw_joint"/>
         <xacro:g1_wheel_joint joint_name="Left_Wheel_Joint"/>
         <xacro:g1_wheel_joint joint_name="Right_Wheel_Joint"/>
+        <!-- Dex3 hands: 7 finger joints each, position-controlled by a per-hand JTC.
+             Order matches the Dex3 motor index order (thumb 0..2, middle 0..1,
+             index 0..1) used by the hardware bridge. -->
+        <xacro:g1_position_joint joint_name="left_hand_thumb_0_joint"/>
+        <xacro:g1_position_joint joint_name="left_hand_thumb_1_joint"/>
+        <xacro:g1_position_joint joint_name="left_hand_thumb_2_joint"/>
+        <xacro:g1_position_joint joint_name="left_hand_middle_0_joint"/>
+        <xacro:g1_position_joint joint_name="left_hand_middle_1_joint"/>
+        <xacro:g1_position_joint joint_name="left_hand_index_0_joint"/>
+        <xacro:g1_position_joint joint_name="left_hand_index_1_joint"/>
+        <xacro:g1_position_joint joint_name="right_hand_thumb_0_joint"/>
+        <xacro:g1_position_joint joint_name="right_hand_thumb_1_joint"/>
+        <xacro:g1_position_joint joint_name="right_hand_thumb_2_joint"/>
+        <xacro:g1_position_joint joint_name="right_hand_middle_0_joint"/>
+        <xacro:g1_position_joint joint_name="right_hand_middle_1_joint"/>
+        <xacro:g1_position_joint joint_name="right_hand_index_0_joint"/>
+        <xacro:g1_position_joint joint_name="right_hand_index_1_joint"/>
       </ros2_control>
     </xacro:unless>

File: src/fm_control/urdf/g1.sim.urdf.xacro (robot description, xacro)
@@ -5,8 +5,8 @@
 This merges the vendored Unitree G1-D geometry (the flat URDF installed into
 fm_description's share) and injects a <ros2_control> system that actuates the 14
-arm joints (7 per arm) plus the two drive wheels, selected by `sim_backend`. The
-waist, legs, and hands are not actuated here — in sim they hold at zero through
-robot_state_publisher. The G1-D is a single fixed configuration, so there is no
-preset arg.
+arm joints (7 per arm), the 14 Dex3 hand joints (7 per hand), and the two drive
+wheels, selected by `sim_backend`. The waist and legs are not actuated here — in sim
+they hold at zero through robot_state_publisher. The G1-D is a single fixed
+configuration, so there is no preset arg.
 For sim_backend=real no ros2_control is emitted: the Servo->arm_sdk bridge drives the
 arm out-of-band (see g1.ros2_control.xacro). The description stays geometry-only so
